Commit message: added front laser to scan ranges in angualar bounds from -PI/4 to PI/4

File: src/mybot_description/urdf/mybot.xacro (robot description, xacro)
@@ -26,69 +26,80 @@
       <origin xyz="0 0 ${wheelRadius}" rpy="0 0 0"/>
       <geometry>
-	<box size="${chassisLength} ${chassisWidth} ${chassisHeight}"/>
-      </geometry>
-    </collision>
-    <visual>
-      <origin xyz="0 0 ${wheelRadius}" rpy="0 0 0"/>
-      <geometry>
-	<box size="${chassisLength} ${chassisWidth} ${chassisHeight}"/>
-      </geometry>
-      <material name="orange"/>
-    </visual>
-    <inertial>
-      <origin xyz="0 0 ${wheelRadius}" rpy="0 0 0"/>
-      <mass value="${chassisMass}"/>
-      <box_inertia m="${chassisMass}" x="${chassisLength}" y="${chassisWidth}" z="${chassisHeight}"/>
-    </inertial>
-  </link>
-  <joint name="fixed" type="fixed">
-    <parent link="chassis"/>
-    <child link="caster_wheel"/>
+       <box size="${chassisLength} ${chassisWidth} ${chassisHeight}"/>
+     </geometry>
+   </collision>
+   <visual>
+    <origin xyz="0 0 ${wheelRadius}" rpy="0 0 0"/>
+    <geometry>
+     <box size="${chassisLength} ${chassisWidth} ${chassisHeight}"/>
+   </geometry>
+   <material name="orange"/>
+ </visual>
+ <inertial>
+  <origin xyz="0 0 ${wheelRadius}" rpy="0 0 0"/>
+  <mass value="${chassisMass}"/>
+  <box_inertia m="${chassisMass}" x="${chassisLength}" y="${chassisWidth}" z="${chassisHeight}"/>
+</inertial>
+</link>
+<joint name="fixed" type="fixed">
+  <parent link="chassis"/>
+  <child link="caster_wheel"/>
+</joint>
+<link name="caster_wheel">
+  <collision>
+    <origin xyz="${casterRadius-chassisLength/2} 0 ${casterRadius-chassisHeight+wheelRadius}" rpy="0 0 0"/>
+    <geometry>
+     <sphere radius="${casterRadius}"/>
+   </geometry>
+ </collision>
+ <visual>
+  <origin xyz="${casterRadius-chassisLength/2} 0 ${casterRadius-chassisHeight+wheelRadius}" rpy="0 0 0"/>
+  <geometry>
+   <sphere radius="${casterRadius}"/>
+ </geometry>
+</visual>
+<inertial>
+  <origin xyz="${casterRadius-chassisLength/2} 0 ${casterRadius-chassisHeight+wheelRadius}" rpy="0 0 0"/>
+  <mass value="${casterMass}"/>
+  <sphere_inertia m="${casterMass}" r="${casterRadius}"/>
+</inertial>
+</link>
+<wheel lr="left" tY="-1"/>
+<wheel lr="right" tY="1"/>
+<joint name="camera_joint" type="fixed">
+  <origin xyz="${-cameraSize+chassisLength/2} 0 ${cameraSize+wheelRadius+cameraSize/2}" rpy="0 0 0"/>
+  <parent link="chassis"/>
+  <child link="camera"/>
+</joint>
+<link name="camera">
+  <collision>
+    <origin xyz="0 0 0" rpy="0 0 0"/>
+    <geometry>
+     <box size="${cameraSize} ${cameraSize} ${cameraSize}"/>
+   </geometry>
+ </collision>
+ <visual>
+  <origin xyz="0 0 0" rpy="0 0 0"/>
+  <geometry>
+   <box size="${cameraSize} ${cameraSize} ${cameraSize}"/>
+ </geometry>
+ <material name="blue"/>
+</visual>
+<inertial>
+  <mass value="${cameraMass}" />
+  <origin xyz="0 0 0" rpy="0 0 0"/>
+  <box_inertia m="${cameraMass}" x="${cameraSize}" y="${cameraSize}" z="${cameraSize}" />
+</inertial>
+</link>
+<!-- FRONT LASER -->
+<xacro:include filename="$(find mybot_description)/urdf/sick_lms1xx_mount.urdf.xacro" />
+<sick_lms1xx_mount prefix="front"
+ topic="mybot/front_laser/scan"/>
+ <joint name="front_laser_mount_joint" type="fixed">
+  <origin xyz="0 0 0"
+    rpy="0 0 0" />
+    <!--parent link="front_mount" />-->
+    <parent link="camera" />
+    <child link="front_laser_mount" />
   </joint>
-  <link name="caster_wheel">
-    <collision>
-      <origin xyz="${casterRadius-chassisLength/2} 0 ${casterRadius-chassisHeight+wheelRadius}" rpy="0 0 0"/>
-      <geometry>
-	<sphere radius="${casterRadius}"/>
-      </geometry>
-    </collision>
-    <visual>
-      <origin xyz="${casterRadius-chassisLength/2} 0 ${casterRadius-chassisHeight+wheelRadius}" rpy="0 0 0"/>
-      <geometry>
-	<sphere radius="${casterRadius}"/>
-      </geometry>
-    </visual>
-    <inertial>
-      <origin xyz="${casterRadius-chassisLength/2} 0 ${casterRadius-chassisHeight+wheelRadius}" rpy="0 0 0"/>
-      <mass value="${casterMass}"/>
-      <sphere_inertia m="${casterMass}" r="${casterRadius}"/>
-    </inertial>
-  </link>
-  <wheel lr="left" tY="-1"/>
-  <wheel lr="right" tY="1"/>
-  <joint name="camera_joint" type="fixed">
-    <origin xyz="${-cameraSize+chassisLength/2} 0 ${cameraSize+wheelRadius+cameraSize/2}" rpy="0 0 0"/>
-    <parent link="chassis"/>
-    <child link="camera"/>
-  </joint>
-  <link name="camera">
-    <collision>
-      <origin xyz="0 0 0" rpy="0 0 0"/>
-      <geometry>
-	<box size="${cameraSize} ${cameraSize} ${cameraSize}"/>
-      </geometry>
-    </collision>
-    <visual>
-      <origin xyz="0 0 0" rpy="0 0 0"/>
-      <geometry>
-	<box size="${cameraSize} ${cameraSize} ${cameraSize}"/>
-      </geometry>
-      <material name="blue"/>
-    </visual>
-    <inertial>
-      <mass value="${cameraMass}" />
-      <origin xyz="0 0 0" rpy="0 0 0"/>
-      <box_inertia m="${cameraMass}" x="${cameraSize}" y="${cameraSize}" z="${cameraSize}" />
-    </inertial>
-  </link>
 </robot>

File: src/mybot_description/urdf/sick_lms1xx_mount.urdf.xacro (robot description, xacro)
@@ -26,20 +26,22 @@
 -->
 <robot xmlns:xacro="http://ros.org/wiki/xacro">
+  <xacro:property name="cameraSize" value="0.05"/>
+  <xacro:property name="cameraMass" value="0.1"/>
   <xacro:include filename="$(find lms1xx)/urdf/sick_lms1xx.urdf.xacro" />
   <xacro:macro name="sick_lms1xx_mount" params="prefix topic">
     <sick_lms1xx frame="${prefix}_laser" topic="${topic}" />
     <link name="${prefix}_laser_mount">
-      <visual>
+      <!--<visual>
         <origin xyz="0 0 0" rpy="0 0 0" />
         <geometry>
-          <!-- Origin of this mesh is the base of the bracket. -->
           <mesh filename="package://jackal_description/meshes/sick-lms1xx-bracket.stl" />
         </geometry>
         <material name="dark_grey" />
-      </visual>
+      </visual>-->
     </link>
     <joint name="${prefix}_laser_joint" type="fixed">
       <!-- This offset is from the base of the bracket to the LIDAR's focal point. -->
-      <origin xyz="0 0 0.149" rpy="0 0 0" />
+      <!--<origin xyz="0 0 0.149" rpy="0 0 0" />-->
+      <origin xyz="0 0 0" rpy="0 0 0" />
       <parent link="${prefix}_laser_mount" />
       <child link="${prefix}_laser" />

Commit message: added arg option for wheel size: e.g. roslaunch [...] wheelRadius:=0.1 wheelWidth:=0.05

File: src/mybot_description/urdf/mybot.xacro (robot description, xacro)
@@ -6,14 +6,17 @@
   <xacro:property name="chassisWidth" value="0.2"/>
   <xacro:property name="chassisMass" value="50"/>
-  <xacro:property name="casterRadius" value="0.05"/>
-  <xacro:property name="casterMass" value="5"/>
-  <xacro:property name="wheelWidth" value="0.05"/>
-  <xacro:property name="wheelRadius" value="0.1"/>
+  <xacro:arg name="wheelWidth" default="0.05" />
+  <xacro:arg name="wheelRadius" default="0.1" />
+  <xacro:property name="wheelWidth" value="$(arg wheelWidth)"/>
+  <xacro:property name="wheelRadius" value="$(arg wheelRadius)"/>
   <xacro:property name="wheelPos" value="0.2"/>
-  <xacro:property name="wheelMass" value="5"/>
+  <!-- calculates the mass of a wheel using the mass density from sample project -->
+  <xacro:property name="wheelMass" value="${10000 * wheelRadius * wheelRadius * wheelWidth}"/>
+  <xacro:property name="casterRadius" value="${wheelRadius - chassisHeight / 2}"/>
+  <!-- calculates the mass of the caster wheel using the mass density from sample project -->
+  <xacro:property name="casterMass" value="${40000 * casterRadius * casterRadius * casterRadius}"/>
   <xacro:property name="cameraSize" value="0.05"/>
   <xacro:property name="cameraMass" value="0.1"/>
-  <xacro:arg name="robot_color" default="Orange" />
-  <xacro:property name="gazebo_robot_color" value="$(arg robot_color)" />
+  <xacro:arg name="robot_color" default="Orange"/>
   <xacro:include filename="$(find mybot_description)/urdf/mybot.gazebo" />
   <xacro:include filename="$(find mybot_description)/urdf/materials.xacro" />
@@ -50,5 +53,6 @@
 <link name="caster_wheel">
   <collision>
-    <origin xyz="${casterRadius-chassisLength/2} 0 ${casterRadius-chassisHeight+wheelRadius}" rpy="0 0 0"/>
+    <!--<origin xyz="${casterRadius-chassisLength/2} 0 ${casterRadius-chassisHeight+wheelRadius}" rpy="0 0 0"/>-->
+    <origin xyz="${casterRadius-chassisLength/2} 0 ${casterRadius}" rpy="0 0 0"/>
     <geometry>
      <sphere radius="${casterRadius}"/>
@@ -56,5 +60,6 @@
  </collision>
  <visual>
-  <origin xyz="${casterRadius-chassisLength/2} 0 ${casterRadius-chassisHeight+wheelRadius}" rpy="0 0 0"/>
+  <!--<origin xyz="${casterRadius-chassisLength/2} 0 ${casterRadius-chassisHeight+wheelRadius}" rpy="0 0 0"/>-->
+    <origin xyz="${casterRadius-chassisLength/2} 0 ${casterRadius}" rpy="0 0 0"/>
   <geometry>
    <sphere radius="${casterRadius}"/>
@@ -62,5 +67,6 @@
 </visual>
 <inertial>
-  <origin xyz="${casterRadius-chassisLength/2} 0 ${casterRadius-chassisHeight+wheelRadius}" rpy="0 0 0"/>
+  <!--<origin xyz="${casterRadius-chassisLength/2} 0 ${casterRadius-chassisHeight+wheelRadius}" rpy="0 0 0"/>-->
+    <origin xyz="${casterRadius-chassisLength/2} 0 ${casterRadius}" rpy="0 0 0"/>
   <mass value="${casterMass}"/>
   <sphere_inertia m="${casterMass}" r="${casterRadius}"/>

Commit message: refactoring and adapted README

File: src/mybot_description/urdf/mybot.xacro (robot description, xacro)
@@ -107,5 +107,4 @@
   <origin xyz="0 0 0"
     rpy="0 0 0" />
-    <!--parent link="front_mount" />-->
     <parent link="camera" />
     <child link="front_laser_mount" />

File: src/mybot_description/urdf/sick_lms1xx_mount.urdf.xacro (robot description, xacro)
@@ -26,6 +26,6 @@
 -->
 <robot xmlns:xacro="http://ros.org/wiki/xacro">
-  <xacro:property name="cameraSize" value="0.05"/>
-  <xacro:property name="cameraMass" value="0.1"/>
+  <!--<xacro:property name="cameraSize" value="0.05"/>
+  <xacro:property name="cameraMass" value="0.1"/>-->
   <xacro:include filename="$(find lms1xx)/urdf/sick_lms1xx.urdf.xacro" />
   <xacro:macro name="sick_lms1xx_mount" params="prefix topic">
